File: BIDIR_5V/BIDIR-5V.kicad_sch (KiCad schematic)
At the start: 16 parts, among them U1 SN74LVC1T45DCK

Commit message: correction cartouche
Other:
- company: Style And Design -> (none)
- title: Module OUT 1 5V -> BIDIR 5V
Changed lines of the file:
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@@
 	(paper "A4")
 	(title_block
-		(title "Module OUT 1 5V")
-		(date "2024-03-04")
-		(rev "00")
-		(company "Style And Design")
-		(comment 1 "T.ORLANDI")
+		(title "BIDIR 5V")
+		(date "2024-12-03")
+		(rev "0")
 	)
 	(junction

Commit message: BIDIR : passage à kicad 9
Changed lines of the file:
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@@
 (kicad_sch
-	(version 20231120)
+	(version 20250114)
 	(generator "eeschema")
-	(generator_version "8.0")
+	(generator_version "9.0")
 	(paper "A4")
 	(title_block
@@
 		(rev "0")
 	)
+	(text "Texas Instruments\nSN74LVC1T45DCKR\nC9382 \n"
+		(exclude_from_sim no)
+		(at 165.1 35.56 0)
+		(effects
+			(font
+				(size 1.27 1.27)
+			)
+			(justify left bottom)
+		)
+	)
+	(text "tension entre 1.65V et 5.5V\n"
+		(exclude_from_sim no)
+		(at 158.75 40.64 0)
+		(effects
+			(font
+				(size 1.27 1.27)
+			)
+			(justify left bottom)
+		)
+	)
+	(text "dir = VCCA <=> A to B"
+		(exclude_from_sim no)
+		(at 160.02 76.2 0)
+		(effects
+			(font
+				(size 1.27 1.27)
+			)
+			(justify left bottom)
+		)
+	)
+	(text "dir = gnd <=> B to A"
+		(exclude_from_sim no)
+		(at 160.02 72.39 0)
+		(effects
+			(font
+				(size 1.27 1.27)
+			)
+			(justify left bottom)
+		)
+	)
 	(junction
 		(at 154.94 60.96)
@@
 		)
 	)
-	(text "Texas Instruments\nSN74LVC1T45DCKR\nC9382 \n"
-		(exclude_from_sim no)
-		(at 165.1 35.56 0)
-		(effects
-			(font
-				(size 1.27 1.27)
-			)
-			(justify left bottom)
-		)
-	)
-	(text "tension entre 1.65V et 5.5V\n"
-		(exclude_from_sim no)
-		(at 158.75 40.64 0)
-		(effects
-			(font
-				(size 1.27 1.27)
-			)
-			(justify left bottom)
-		)
-	)
-	(text "dir = VCCA <=> A to B"
-		(exclude_from_sim no)
-		(at 160.02 76.2 0)
-		(effects
-			(font
-				(size 1.27 1.27)
-			)
-			(justify left bottom)
-		)
-	)
-	(text "dir = gnd <=> B to A"
-		(exclude_from_sim no)
-		(at 160.02 72.39 0)
-		(effects
-			(font
-				(size 1.27 1.27)
-			)
-			(justify left bottom)
-		)
-	)
 	(label "OUT"
 		(at 86.36 38.1 0)
-		(fields_autoplaced yes)
 		(effects
 			(font
@@
 	(label "5V"
 		(at 176.53 44.45 0)
-		(fields_autoplaced yes)
 		(effects
 			(font
@@
 	(label "GND"
 		(at 128.27 69.85 180)
-		(fields_autoplaced yes)
 		(effects
 			(font
@@
 	(label "5V"
 		(at 59.69 48.26 0)
-		(fields_autoplaced yes)
 		(effects
 			(font
@@
 	(label "3V3"
 		(at 86.36 63.5 0)
-		(fields_autoplaced yes)
 		(effects
 			(font
@@
 	(label "GND"
 		(at 217.17 71.12 0)
-		(fields_autoplaced yes)
 		(effects
 			(font
@@
 	(label "GND"
 		(at 135.89 46.99 180)
-		(fields_autoplaced yes)
 		(effects
 			(font
@@
 	(label "3V3"
 		(at 135.89 36.83 180)
-		(fields_autoplaced yes)
 		(effects
 			(font
@@
 	(label "GND"
 		(at 59.69 67.31 0)
-		(fields_autoplaced yes)
 		(effects
 			(font
@@
 	(label "3V3"
 		(at 168.91 44.45 180)
-		(fields_autoplaced yes)
 		(effects
 			(font
@@
 	(label "GND"
 		(at 196.85 46.99 180)
-		(fields_autoplaced yes)
 		(effects
 			(font
@@
 	(label "OUT_i"
 		(at 110.49 55.88 180)
-		(fields_autoplaced yes)
 		(effects
 			(font
@@
 	(label "GND"
 		(at 171.45 67.31 180)
-		(fields_autoplaced yes)
 		(effects
 			(font
@@
 	(label "OUT"
 		(at 217.17 55.88 0)
-		(fields_autoplaced yes)
 		(effects
 			(font
@@
 	(label "GND"
 		(at 203.2 71.12 0)
-		(fields_autoplaced yes)
 		(effects
 			(font
@@
 	(label "GND"
 		(at 153.67 71.12 180)
-		(fields_autoplaced yes)
 		(effects
 			(font
@@
 	(label "3V3"
 		(at 59.69 58.42 0)
-		(fields_autoplaced yes)
 		(effects
 			(font
@@
 	(label "3V3"
 		(at 139.7 60.96 180)
-		(fields_autoplaced yes)
 		(effects
 			(font
@@
 	(label "GND"
 		(at 114.3 69.85 180)
-		(fields_autoplaced yes)
 		(effects
 			(font
@@
 	(label "GND"
 		(at 86.36 72.39 0)
-		(fields_autoplaced yes)
 		(effects
 			(font
@@
 	(label "OUT_i"
 		(at 86.36 46.99 0)
-		(fields_autoplaced yes)
 		(effects
 			(font
@@
 	(label "5V"
 		(at 86.36 55.88 0)
-		(fields_autoplaced yes)
 		(effects
 			(font
@@
 	(label "5V"
 		(at 196.85 36.83 180)
-		(fields_autoplaced yes)
 		(effects
 			(font
@@
 		)
 	)
+	(embedded_fonts no)
 )

Commit message: retouche pour 10mm de large
Parts:
- added TP6: TestPoint, Chimere_comps:Pastille, symbol Connector:TestPoint
Connections:
- net GND: now also TP6.1
Changed lines of the file:
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@@
+	(wire
+		(pts
+			(xy 81.28 80.01) (xy 86.36 80.01)
+		)
+		(stroke
+			(width 0)
+			(type default)
+		)
+	)
 	(wire
 		(pts
@@
 			)
 			(justify right bottom)
+		)
+	)
+	(label "GND"
+		(at 86.36 80.01 0)
+		(effects
+			(font
+				(size 1.27 1.27)
+			)
+			(justify left bottom)
 		)
 	)
@@
 					(unit 1)
 				)
+			)
+		)
+	)
+	(symbol
+		(lib_id "Connector:TestPoint")
+		(at 81.28 80.01 90)
+		(unit 1)
+		(exclude_from_sim no)
+		(in_bom no)
+		(on_board yes)
+		(dnp no)
+		(fields_autoplaced yes)
+		(property "Reference" "TP6"
+			(at 77.978 74.93 90)
+			(effects
+				(font
+					(size 1.27 1.27)
+				)
+			)
+		)
+		(property "Value" "TestPoint"
+			(at 77.978 77.47 90)
+			(effects
+				(font
+					(size 1.27 1.27)
+				)
+			)
+		)
+		(property "Footprint" "Chimere_comps:Pastille"
+			(at 81.28 74.93 0)
+			(effects
+				(font
+					(size 1.27 1.27)
+				)
+				(hide yes)
+			)
+		)
+		(property "Datasheet" "~"
+			(at 81.28 74.93 0)
+			(effects
+				(font
+					(size 1.27 1.27)
+				)
+				(hide yes)
+			)
+		)
+		(property "Description" ""
+			(at 81.28 80.01 0)
+			(effects
+				(font
+					(size 1.27 1.27)
+				)
+				(hide yes)
+			)
+		)
+		(pin "1"
+		)
+		(instances
+			(project "BIDIR-5V"
+				(path "/e63e39d7-6ac0-4ffd-8aa3-1841a4541b55"
+					(reference "TP6")
+					(unit 1)
+				)
